File: cartridge/pcb/vx_cart_v1.01/vectrex_cart_v1.01.kicad_sch (KiCad schematic)
At the start: 7 parts, among them J1 Vectrex Cartridge Connector, U1 27C256

Commit message: Cart PCB v1.01
Parts:
- R1: value OR -> 0R; footprint Resistor_SMD:R_0402_1005Metric -> Resistor_THT:R_Axial_DIN0204_L3.6mm_D1.6mm_P7.62mm_Horizontal
- R2: footprint Resistor_THT:R_Axial_DIN0204_L3.6mm_D1.6mm_P5.08mm_Horizontal -> Resistor_THT:R_Axial_DIN0204_L3.6mm_D1.6mm_P7.62mm_Horizontal
- U1: footprint Package_DIP:DIP-28_W15.24mm -> Package_DIP:DIP-28_W15.24mm_LongPads
Other:
- title: Vectrex Eprom v1.0 -> Vectrex cartridge PCB
- moved on the sheet: R2
Changed lines of the file:
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@@
 	(paper "A4")
 	(title_block
-		(title "Vectrex Eprom v1.0")
+		(title "Vectrex cartridge PCB")
+		(date "2024-04-18")
+		(rev "v1.01")
 	)
 	(junction
@@
 	)
 	(junction
-		(at 80.01 73.66)
-		(diameter 0)
-		(color 0 0 0 0)
-	)
-	(junction
 		(at 45.72 29.21)
 		(diameter 0)
 		(color 0 0 0 0)
 	)
+	(junction
+		(at 83.82 73.66)
+		(diameter 0)
+		(color 0 0 0 0)
+	)
 	(no_connect
 		(at 38.1 26.67)
@@
 	(wire
 		(pts
-			(xy 74.93 73.66) (xy 80.01 73.66)
-		)
-		(stroke
-			(width 0)
-			(type default)
-		)
-	)
-	(wire
-		(pts
 			(xy 45.72 87.63) (xy 38.1 87.63)
 		)
@@
 	(wire
 		(pts
-			(xy 64.77 78.74) (xy 67.31 78.74)
-		)
-		(stroke
-			(width 0)
-			(type default)
-		)
-	)
-	(wire
-		(pts
 			(xy 128.27 48.26) (xy 139.7 48.26)
 		)
@@
 	(wire
 		(pts
-			(xy 80.01 73.66) (xy 80.01 78.74)
-		)
-		(stroke
-			(width 0)
-			(type default)
-		)
-	)
-	(wire
-		(pts
 			(xy 38.1 82.55) (xy 40.64 82.55)
 		)
@@
 	(wire
 		(pts
+			(xy 83.82 68.58) (xy 83.82 73.66)
+		)
+		(stroke
+			(width 0)
+			(type default)
+		)
+	)
+	(wire
+		(pts
 			(xy 209.55 152.4) (xy 201.93 152.4)
 		)
@@
 	(wire
 		(pts
+			(xy 83.82 73.66) (xy 107.95 73.66)
+		)
+		(stroke
+			(width 0)
+			(type default)
+		)
+	)
+	(wire
+		(pts
 			(xy 93.98 66.04) (xy 107.95 66.04)
 		)
@@
 	(wire
 		(pts
-			(xy 64.77 73.66) (xy 67.31 73.66)
-		)
-		(stroke
-			(width 0)
-			(type default)
-		)
-	)
-	(wire
-		(pts
 			(xy 118.11 88.9) (xy 118.11 99.06)
 		)
@@
 	(wire
 		(pts
+			(xy 76.2 78.74) (xy 83.82 78.74)
+		)
+		(stroke
+			(width 0)
+			(type default)
+		)
+	)
+	(wire
+		(pts
 			(xy 38.1 34.29) (xy 45.72 34.29)
 		)
@@
 	(wire
 		(pts
+			(xy 64.77 78.74) (xy 68.58 78.74)
+		)
+		(stroke
+			(width 0)
+			(type default)
+		)
+	)
+	(wire
+		(pts
+			(xy 64.77 68.58) (xy 68.58 68.58)
+		)
+		(stroke
+			(width 0)
+			(type default)
+		)
+	)
+	(wire
+		(pts
 			(xy 38.1 29.21) (xy 45.72 29.21)
 		)
@@
 	(wire
 		(pts
-			(xy 80.01 73.66) (xy 107.95 73.66)
-		)
-		(stroke
-			(width 0)
-			(type default)
-		)
-	)
-	(wire
-		(pts
 			(xy 38.1 69.85) (xy 40.64 69.85)
 		)
@@
 	(wire
 		(pts
+			(xy 83.82 78.74) (xy 83.82 73.66)
+		)
+		(stroke
+			(width 0)
+			(type default)
+		)
+	)
+	(wire
+		(pts
 			(xy 45.72 29.21) (xy 46.99 29.21)
 		)
@@
 	(wire
 		(pts
+			(xy 76.2 68.58) (xy 83.82 68.58)
+		)
+		(stroke
+			(width 0)
+			(type default)
+		)
+	)
+	(wire
+		(pts
 			(xy 128.27 45.72) (xy 139.7 45.72)
 		)
@@
 	(wire
 		(pts
-			(xy 80.01 78.74) (xy 74.93 78.74)
-		)
-		(stroke
-			(width 0)
-			(type default)
-		)
-	)
-	(wire
-		(pts
 			(xy 40.64 31.75) (xy 38.1 31.75)
 		)
@@
 	(global_label "A14"
 		(shape input)
-		(at 64.77 73.66 180)
+		(at 64.77 68.58 180)
 		(fields_autoplaced yes)
 		(effects
@@
 		)
 		(property "Intersheetrefs" "${INTERSHEET_REFS}"
-			(at 58.9314 73.66 0)
+			(at 58.9314 68.58 0)
 			(effects
 				(font
@@
 		)
 		(instances
-			(project "27C256cart"
+			(project "vectrex_cart_v1.01"
 				(path "/10a0b369-9141-4c8d-bebf-e0e7bbaefd7e"
 					(reference "J1")
@@
 		)
 		(instances
-			(project "27C256cart"
+			(project "vectrex_cart_v1.01"
 				(path "/10a0b369-9141-4c8d-bebf-e0e7bbaefd7e"
 					(reference "H2")
@@
 		)
 		(instances
-			(project "27C256cart"
+			(project "vectrex_cart_v1.01"
 				(path "/10a0b369-9141-4c8d-bebf-e0e7bbaefd7e"
 					(reference "H1")
@@
 		)
 		(instances
-			(project "27C256cart"
+			(project "vectrex_cart_v1.01"
 				(path "/10a0b369-9141-4c8d-bebf-e0e7bbaefd7e"
 					(reference "H3")
@@
 	(symbol
 		(lib_id "Device:R")
-		(at 71.12 73.66 270)
+		(at 72.39 68.58 270)
 		(unit 1)
 		(exclude_from_sim no)
@@
 		(dnp no)
 		(property "Reference" "R1"
-			(at 71.12 71.628 90)
-			(effects
-				(font
-					(size 1.27 1.27)
-				)
-			)
-		)
-		(property "Value" "OR"
-			(at 71.12 73.914 90)
-			(effects
-				(font
-					(size 1.27 1.27)
-				)
-			)
-		)
-		(property "Footprint" "Resistor_SMD:R_0402_1005Metric"
-			(at 71.12 71.882 90)
+			(at 72.39 66.548 90)
+			(effects
+				(font
+					(size 1.27 1.27)
+				)
+			)
+		)
+		(property "Value" "0R"
+			(at 72.39 68.834 90)
+			(effects
+				(font
+					(size 1.27 1.27)
+				)
+			)
+		)
+		(property "Footprint" "Resistor_THT:R_Axial_DIN0204_L3.6mm_D1.6mm_P7.62mm_Horizontal"
+			(at 72.39 66.802 90)
 			(effects
 				(font
@@
 		)
 		(property "Datasheet" "~"
-			(at 71.12 73.66 0)
+			(at 72.39 68.58 0)
 			(effects
 				(font
@@
 		)
 		(property "Description" "Resistor"
-			(at 71.12 73.66 0)
+			(at 72.39 68.58 0)
 			(effects
 				(font
@@
 		)
 		(instances
-			(project "27C256cart"
+			(project "vectrex_cart_v1.01"
 				(path "/10a0b369-9141-4c8d-bebf-e0e7bbaefd7e"
 					(reference "R1")
@@
 		)
 		(instances
-			(project "27C256cart"
+			(project "vectrex_cart_v1.01"
 				(path "/10a0b369-9141-4c8d-bebf-e0e7bbaefd7e"
 					(reference "#PWR0102")
@@
 		)
 		(instances
-			(project "27C256cart"
+			(project "vectrex_cart_v1.01"
 				(path "/10a0b369-9141-4c8d-bebf-e0e7bbaefd7e"
 					(reference "#PWR0101")
@@
 		)
 		(instances
-			(project "27C256cart"
+			(project "vectrex_cart_v1.01"
 				(path "/10a0b369-9141-4c8d-bebf-e0e7bbaefd7e"
 					(reference "#FLG0102")
@@
 		)
 		(instances
-			(project "27C256cart"
+			(project "vectrex_cart_v1.01"
 				(path "/10a0b369-9141-4c8d-bebf-e0e7bbaefd7e"
 					(reference "#FLG0101")
@@
 	(symbol
 		(lib_id "Device:R")
-		(at 71.12 78.74 270)
+		(at 72.39 78.74 270)
 		(unit 1)
 		(exclude_from_sim no)
@@
 		(dnp no)
 		(property "Reference" "R2"
-			(at 71.12 76.708 90)
+			(at 72.39 76.708 90)
 			(effects
 				(font
@@
 		)
 		(property "Value" "1K"
-			(at 71.12 78.994 90)
-			(effects
-				(font
-					(size 1.27 1.27)
-				)
-			)
-		)
-		(property "Footprint" "Resistor_THT:R_Axial_DIN0204_L3.6mm_D1.6mm_P5.08mm_Horizontal"
-			(at 71.12 76.962 90)
+			(at 72.39 78.994 90)
+			(effects
+				(font
+					(size 1.27 1.27)
+				)
+			)
+		)
+		(property "Footprint" "Resistor_THT:R_Axial_DIN0204_L3.6mm_D1.6mm_P7.62mm_Horizontal"
+			(at 72.39 76.962 90)
 			(effects
 				(font
@@
 		)
 		(property "Datasheet" "~"
-			(at 71.12 78.74 0)
+			(at 72.39 78.74 0)
 			(effects
 				(font
@@
 		)
 		(property "Description" "Resistor"
-			(at 71.12 78.74 0)
+			(at 72.39 78.74 0)
 			(effects
 				(font
@@
 		)
 		(instances
-			(project "27C256cart"
+			(project "vectrex_cart_v1.01"
 				(path "/10a0b369-9141-4c8d-bebf-e0e7bbaefd7e"
 					(reference "R2")
@@
 			)
 		)
-		(property "Footprint" "Package_DIP:DIP-28_W15.24mm"
+		(property "Footprint" "Package_DIP:DIP-28_W15.24mm_LongPads"
 			(at 118.11 60.96 0)
 			(effects
@@
 		)
 		(instances
-			(project "27C256cart"
+			(project "vectrex_cart_v1.01"
 				(path "/10a0b369-9141-4c8d-bebf-e0e7bbaefd7e"
 					(reference "U1")
